File: KiCad/#2_7Segment/#2_7segment.kicad_pcb (KiCad board)
At the start: 2 copper layers, 52.3 x 21.5 mm, 11 parts, among them J1 Conn_02x19_Odd_Even, U1 7 segment display

Commit message: Silk screen
Parts:
- added REF**: OSHW-Logo2_7.3x6mm_SilkScreen, Symbol:OSHW-Logo2_7.3x6mm_SilkScreen, B.Cu at (172.8, 105.7)
